File: debug.sch (KiCad schematic (older format))
At the start: 56 parts

Commit message: progress
Parts:
- removed U? (x3): NTSX2102GU8H, symbol NTSX2102GU8H
- added D2, D4: TVS, footprints:D_0603, symbol TVS
- added R10: 0, Resistors_SMD:R_0603_HandSoldering, symbol R
- added U2, U3, U7: NLSX4373DR2G, footprints:SO-8, symbol NLSX4373DR2G
- C1, C10, C11, C12, C13, C14, C15, C2, C3, C4, C5, C6, C7, C8, C9: renamed from C?; footprint (none) -> Capacitors_SMD:C_0603_HandSoldering
- D1, D3, D5: renamed from D?; footprint (none) -> footprints:D_0603
- D7: renamed from D?; footprint (none) -> Diodes_SMD:SOD-523
- FB1, FB2: renamed from FB?; footprint (none) -> footprints:L_0603
- J1: renamed from P?; footprint (none) -> Connect:USB_Mini-B
- J2, J6: renamed from P?; footprint (none) -> Pin_Headers:Pin_Header_Straight_1x04
- JP1: renamed from JP?; footprint (none) -> Pin_Headers:Pin_Header_Straight_1x03
- JP2: renamed from JP?; footprint (none) -> Pin_Headers:Pin_Header_Straight_1x02
- Q1, Q2, Q3: renamed from Q?; footprint (none) -> TO_SOT_Packages_SMD:SOT-23_Handsoldering
- R1, R2, R3, R4, R5, R6, R7, R8, R9: renamed from R?; footprint (none) -> Resistors_SMD:R_0603_HandSoldering
- SW1, SW2, SW3: renamed from SW?; footprint (none) -> footprints:PTS645SM43SMTR92
- U1: renamed from U?; footprint (none) -> SMD_Packages:SSOP-14
- U4: renamed from U?; footprint SOT-223 -> TO_SOT_Packages_SMD:SOT-223
- U5: renamed from U?; footprint QFN32 -> (none)
- U6: renamed from U?; footprint (none) -> SMD_Packages:SOIC-8-N
- gave numbers to parts that had none: 6
Connections:
- wire segments 201 -> 204
- no-connect marks 11 -> 13
Other:
- moved on the sheet: C4, J4, J6, JP2, R4, SW2

Commit message: more progress
Parts:
- D6: footprint (none) -> footprints:PLCC4
- J3, J4: footprint (none) -> footprints:FTSH-105-01-L-DV-K
Changed lines of the file:
@@
 F 0 "J4" H 5700 9400 50  0000 C CNN
 F 1 "TARGET_DEBUG" H 5700 8800 50  0000 C CNN
-F 2 "" H 5700 7900 50  0001 C CNN
+F 2 "footprints:FTSH-105-01-L-DV-K" H 5700 7900 50  0001 C CNN
 F 3 "" H 5700 7900 50  0000 C CNN
 	1    5700 9100
@@
 F 0 "J3" H 5400 1850 50  0000 C CNN
 F 1 "DEBUG" H 5400 1250 50  0000 C CNN
-F 2 "" H 5400 350 50  0001 C CNN
+F 2 "footprints:FTSH-105-01-L-DV-K" H 5400 350 50  0001 C CNN
 F 3 "" H 5400 350 50  0000 C CNN
 	1    5400 1550
@@
 F 0 "D6" H 15350 5850 50  0000 C CNN
 F 1 "Led_RGB_CA" H 15350 5150 50  0000 C CNN
-F 2 "" H 15305 5450 50  0001 C CNN
+F 2 "footprints:PLCC4" H 15305 5450 50  0001 C CNN
 F 3 "" H 15305 5450 50  0000 C CNN
 	1    15350 5500

Commit message: more progress
Parts:
- added R11: 0, Resistors_SMD:R_0603_HandSoldering, symbol R
- J5: footprint (none) -> footprints:SD-105027-001
- U5: footprint (none) -> footprints:MK20DX128VFM5
- Y1: footprint (none) -> footprints:FX135
- Y2: footprint (none) -> Crystals:Crystal_SMD_5032_4Pads
Connections:
- wire segments 204 -> 206
Other:
- note added: "DNP"
Changed lines of the file:
@@
 F 0 "J5" H 14800 1200 60  0000 C CNN
 F 1 "MOLEX-MICRO-SD" H 14850 2350 60  0000 C CNN
-F 2 "" H 14800 1000 60  0001 C CNN
+F 2 "footprints:SD-105027-001" H 14800 1000 60  0001 C CNN
 F 3 "" H 14800 1000 60  0001 C CNN
 	1    14850 1750
@@
 F 0 "Y1" V 9400 8750 50  0000 C CNN
 F 1 "32KHz" H 9400 8450 50  0000 C CNN
-F 2 "" H 9400 8600 50  0001 C CNN
+F 2 "footprints:FX135" H 9400 8600 50  0001 C CNN
 F 3 "" H 9400 8600 50  0000 C CNN
 	1    9400 8600
@@
 F 0 "Y2" V 9400 9600 50  0000 C CNN
 F 1 "8MHz" H 9400 9300 50  0000 C CNN
-F 2 "" H 9400 9450 50  0001 C CNN
+F 2 "Crystals:Crystal_SMD_5032_4Pads" H 9400 9450 50  0001 C CNN
 F 3 "" H 9400 9450 50  0000 C CNN
 	1    9400 9450
@@
 F 0 "U5" H 8450 6850 50  0000 L CNN
 F 1 "MK20DX128VFM5" H 8700 4350 50  0000 L CNN
-F 2 "" H 10000 4800 50  0001 L CNN
+F 2 "footprints:MK20DX128VFM5" H 10000 4800 50  0001 L CNN
 F 3 "MCU 32-bit Kinetis K20 ARM Cortex M4 RISC 128KB Flash 1.8V/2.5V/3.3V 32-Pin QFN Tray" H 10000 5600 50  0001 L CNN
 F 4 "Freescale Semiconductor" H 10000 5250 50  0001 L CNN "MF"
@@
 	14250 4700 14350 4700
 Wire Wire Line
-	15650 5500 15650 5400
-Wire Wire Line
-	15550 5500 15650 5500
+	15650 5400 15650 5750
+Wire Wire Line
+	15550 5500 15800 5500
 Wire Wire Line
 	14250 5200 14350 5200
@@
 L D_Schottky D7
 U 1 1 58107630
-P 15800 5500
-F 0 "D7" H 15800 5600 50  0000 C CNN
-F 1 "D_Schottky" H 15800 5400 50  0000 C CNN
-F 2 "Diodes_SMD:SOD-523" H 15800 5500 50  0001 C CNN
-F 3 "" H 15800 5500 50  0000 C CNN
-	1    15800 5500
+P 15950 5500
+F 0 "D7" H 15950 5600 50  0000 C CNN
+F 1 "D_Schottky" H 15950 5400 50  0000 C CNN
+F 2 "Diodes_SMD:SOD-523" H 15950 5500 50  0001 C CNN
+F 3 "" H 15950 5500 50  0000 C CNN
+	1    15950 5500
 	1    0    0    -1
 $EndComp
@@
 L VCC #PWR047
 U 1 1 58107BD2
-P 16050 5400
-F 0 "#PWR047" H 16050 5250 50  0001 C CNN
-F 1 "VCC" H 16050 5550 50  0000 C CNN
-F 2 "" H 16050 5400 50  0000 C CNN
-F 3 "" H 16050 5400 50  0000 C CNN
-	1    16050 5400
-	1    0    0    -1
-$EndComp
-Wire Wire Line
-	15950 5500 16050 5500
-Wire Wire Line
-	16050 5500 16050 5400
+P 16200 5400
+F 0 "#PWR047" H 16200 5250 50  0001 C CNN
+F 1 "VCC" H 16200 5550 50  0000 C CNN
+F 2 "" H 16200 5400 50  0000 C CNN
+F 3 "" H 16200 5400 50  0000 C CNN
+	1    16200 5400
+	1    0    0    -1
+$EndComp
+Wire Wire Line
+	16100 5500 16200 5500
+Wire Wire Line
+	16200 5400 16200 5750
 $Comp
 L TVS D2
@@
 Wire Wire Line
 	15650 5000 15650 5100
+$Comp
+L R R11
+U 1 1 581DFAB0
+P 15950 5750
+F 0 "R11" V 16030 5750 50  0000 C CNN
+F 1 "0" V 15950 5750 50  0000 C CNN
+F 2 "Resistors_SMD:R_0603_HandSoldering" V 15880 5750 50  0001 C CNN
+F 3 "" H 15950 5750 50  0000 C CNN
+	1    15950 5750
+	0    1    1    0
+$EndComp
+Connection ~ 15650 5500
+Wire Wire Line
+	15650 5750 15800 5750
+Wire Wire Line
+	16200 5750 16100 5750
+Connection ~ 16200 5500
+Text Notes 16050 5850 0    60   ~ 0
+DNP
 $EndSCHEMATC

Commit message: minor sch tweaks, starting to route (poorly)
Parts:
- removed Y2: 8MHz, Crystals:Crystal_SMD_5032_4Pads, symbol Crystal
- added Y2: 8MHz, Crystals:Crystal_SMD_5032_4Pads, symbol CRYSTAL_SMD
- Q1, Q2, Q3: footprint TO_SOT_Packages_SMD:SOT-23_Handsoldering -> TO_SOT_Packages_SMD:SOT-23
Connections:
- net labels added: USB2_D+, USB2_D-, USB_D+, USB_D-
- net labels removed: USB_DM, USB_DP
- wire segments 206 -> 207
Other:
- moved on the sheet: C13
Changed lines of the file:
@@
 $EndComp
 Text GLabel 3050 2200 2    60   Input ~ 0
-USB_DM
+USB2_D-
 Text GLabel 3050 2300 2    60   Input ~ 0
-USB_DP
+USB2_D+
 NoConn ~ 1450 2400
 Text GLabel 10150 5250 2    60   Input ~ 0
@@
 F 3 "" H 9400 8600 50  0000 C CNN
 	1    9400 8600
-	0    1    1    0
-$EndComp
-$Comp
-L Crystal Y2
-U 1 1 580C5D3A
-P 9400 9450
-F 0 "Y2" V 9400 9600 50  0000 C CNN
-F 1 "8MHz" H 9400 9300 50  0000 C CNN
-F 2 "Crystals:Crystal_SMD_5032_4Pads" H 9400 9450 50  0001 C CNN
-F 3 "" H 9400 9450 50  0000 C CNN
-	1    9400 9450
 	0    1    1    0
 $EndComp
@@
 	1    0    0    -1
 $EndComp
-Text GLabel 8150 4950 0    60   Input ~ 0
-USB_DP
-Text GLabel 8150 4850 0    60   Input ~ 0
-USB_DM
 $Comp
 L C C5
@@
 L C C13
 U 1 1 580DC92F
-P 9000 9600
-F 0 "C13" H 9025 9700 50  0000 L CNN
-F 1 "C" V 9050 9500 50  0000 L CNN
-F 2 "Capacitors_SMD:C_0603_HandSoldering" H 9038 9450 50  0001 C CNN
-F 3 "" H 9000 9600 50  0000 C CNN
-	1    9000 9600
+P 9000 9700
+F 0 "C13" H 9025 9800 50  0000 L CNN
+F 1 "C" V 9050 9600 50  0000 L CNN
+F 2 "Capacitors_SMD:C_0603_HandSoldering" H 9038 9550 50  0001 C CNN
+F 3 "" H 9000 9700 50  0000 C CNN
+	1    9000 9700
 	0    1    1    0
 $EndComp
@@
 L GND #PWR043
 U 1 1 580DCC0D
-P 8750 9600
-F 0 "#PWR043" H 8750 9350 50  0001 C CNN
-F 1 "GND" H 8750 9450 50  0000 C CNN
-F 2 "" H 8750 9600 50  0000 C CNN
-F 3 "" H 8750 9600 50  0000 C CNN
-	1    8750 9600
+P 8750 9700
+F 0 "#PWR043" H 8750 9450 50  0001 C CNN
+F 1 "GND" H 8750 9550 50  0000 C CNN
+F 2 "" H 8750 9700 50  0000 C CNN
+F 3 "" H 8750 9700 50  0000 C CNN
+	1    8750 9700
 	-1   0    0    -1
 $EndComp
@@
 F 0 "Q1" V 14600 5000 50  0000 R CNN
 F 1 "Q_NMOS_DGS" V 14250 5500 50  0000 R CNN
-F 2 "TO_SOT_Packages_SMD:SOT-23_Handsoldering" H 14550 5000 50  0001 C CNN
+F 2 "TO_SOT_Packages_SMD:SOT-23" H 14550 5000 50  0001 C CNN
 F 3 "" H 14350 4900 50  0000 C CNN
 	1    14350 4900
@@
 F 0 "Q2" V 14600 5500 50  0000 R CNN
 F 1 "Q_NMOS_DGS" V 14350 5250 50  0000 R CNN
-F 2 "TO_SOT_Packages_SMD:SOT-23_Handsoldering" H 14550 5500 50  0001 C CNN
+F 2 "TO_SOT_Packages_SMD:SOT-23" H 14550 5500 50  0001 C CNN
 F 3 "" H 14350 5400 50  0000 C CNN
 	1    14350 5400
@@
 F 0 "Q3" V 14600 6000 50  0000 R CNN
 F 1 "Q_NMOS_DGS" V 14350 5750 50  0000 R CNN
-F 2 "TO_SOT_Packages_SMD:SOT-23_Handsoldering" H 14550 6000 50  0001 C CNN
+F 2 "TO_SOT_Packages_SMD:SOT-23" H 14550 6000 50  0001 C CNN
 F 3 "" H 14350 5900 50  0000 C CNN
 	1    14350 5900
@@
 Text GLabel 8150 5950 0    60   Input ~ 0
 EXTAL
-Text GLabel 9650 9300 2    60   Input ~ 0
+Text GLabel 9650 8450 2    60   Input ~ 0
 XTAL32
-Text GLabel 9650 9600 2    60   Input ~ 0
+Text GLabel 9650 8750 2    60   Input ~ 0
 EXTAL32
-Text GLabel 9650 8450 2    60   Input ~ 0
+Text GLabel 9750 9300 2    60   Input ~ 0
 XTAL
-Text GLabel 9650 8750 2    60   Input ~ 0
+Text GLabel 9750 9700 2    60   Input ~ 0
 EXTAL
 Text Notes 9000 9100 0    120  ~ 0
@@
 	8100 6150 8250 6150
 Wire Wire Line
-	9150 9600 9650 9600
-Wire Wire Line
-	9150 9300 9650 9300
+	9150 9700 9750 9700
+Wire Wire Line
+	9150 9300 9750 9300
 Wire Wire Line
 	9150 8750 9650 8750
@@
 	8850 8450 8850 8750
 Wire Wire Line
-	8850 9300 8850 9600
+	8850 9300 8850 9700
 Connection ~ 9400 9300
-Connection ~ 9400 9600
-Wire Wire Line
-	8850 9600 8750 9600
+Connection ~ 9400 9700
+Wire Wire Line
+	8850 9700 8750 9700
 Wire Wire Line
 	8850 8750 8750 8750
@@
 Text Notes 16050 5850 0    60   ~ 0
 DNP
+$Comp
+L CRYSTAL_SMD Y2
+U 1 1 581E7BB6
+P 9400 9500
+F 0 "Y2" H 9400 9590 50  0000 C CNN
+F 1 "8MHz" H 9300 9700 50  0000 L CNN
+F 2 "Crystals:Crystal_SMD_5032_4Pads" H 9400 9500 50  0001 C CNN
+F 3 "" H 9400 9500 50  0000 C CNN
+	1    9400 9500
+	0    -1   -1   0
+$EndComp
+$Comp
+L GND #PWR048
+U 1 1 581E840C
+P 9600 9500
+F 0 "#PWR048" H 9600 9250 50  0001 C CNN
+F 1 "GND" H 9600 9350 50  0000 C CNN
+F 2 "" H 9600 9500 50  0000 C CNN
+F 3 "" H 9600 9500 50  0000 C CNN
+	1    9600 9500
+	-1   0    0    -1
+$EndComp
+Wire Wire Line
+	9500 9500 9600 9500
+$Comp
+L VCC #PWR049
+U 1 1 581E985E
+P 7700 4650
+F 0 "#PWR049" H 7700 4500 50  0001 C CNN
+F 1 "VCC" H 7700 4800 50  0000 C CNN
+F 2 "" H 7700 4650 50  0000 C CNN
+F 3 "" H 7700 4650 50  0000 C CNN
+	1    7700 4650
+	1    0    0    -1
+$EndComp
+Connection ~ 7700 4650
+Text Label 2200 2200 0    60   ~ 0
+USB_D-
+Text Label 2200 2300 0    60   ~ 0
+USB_D+
+Text GLabel 8150 4850 0    60   Input ~ 0
+USB2_D-
+Text GLabel 8150 4950 0    60   Input ~ 0
+USB2_D+
 $EndSCHEMATC

Commit message: replace large components with smaller ones
change to simple switching power supply
add board outline
simplify USB protection
Parts:
- removed D1, D3, D5: TVS, footprints:D_0603, symbol TVS
- removed JP1: JUMPER3, Pin_Headers:Pin_Header_Straight_1x03, symbol JUMPER3
- removed R2, R3: 33, Resistors_SMD:R_0603_HandSoldering, symbol R
- removed U2, U3, U7: NLSX4373DR2G, footprints:SO-8, symbol NLSX4373DR2G
- removed U4: TC1262-33VDB, TO_SOT_Packages_SMD:SOT-223, symbol TC1262-33VDB
- added L1: 2.2 uH, footprints:1008, symbol INDUCTOR
- added R6, R7: 0, Resistors_SMD:R_0603, symbol R
- added U2: FXMA108BQX, footprints:DQFN20, symbol FXMA108BQX
- added U3: PAM2301, TO_SOT_Packages_SMD:SOT-23-5, symbol PAM2301
- added U?: STF202-22, symbol STF202-22
- C1: renamed from C2; footprint Capacitors_SMD:C_0603_HandSoldering -> Capacitors_SMD:C_0603
- C10: renamed from C14; footprint Capacitors_SMD:C_0603_HandSoldering -> Capacitors_SMD:C_0603
- C11: renamed from C15; footprint Capacitors_SMD:C_0603_HandSoldering -> Capacitors_SMD:C_0603
- C12: renamed from C10; footprint Capacitors_SMD:C_0603_HandSoldering -> Capacitors_SMD:C_0603
- C13: renamed from C11; footprint Capacitors_SMD:C_0603_HandSoldering -> Capacitors_SMD:C_0603
- C14: renamed from C12; footprint Capacitors_SMD:C_0603_HandSoldering -> Capacitors_SMD:C_0603
- C15: renamed from C13; footprint Capacitors_SMD:C_0603_HandSoldering -> Capacitors_SMD:C_0603
- C2: renamed from C5; footprint Capacitors_SMD:C_0603_HandSoldering -> Capacitors_SMD:C_0603
- C3: renamed from C6; footprint Capacitors_SMD:C_0603_HandSoldering -> Capacitors_SMD:C_0603
- C4: renamed from C7; footprint Capacitors_SMD:C_0603_HandSoldering -> Capacitors_SMD:C_0603
- C5: renamed from C1; value 1u -> 10u; footprint Capacitors_SMD:C_0603_HandSoldering -> Capacitors_SMD:C_0603
- C6: renamed from C4; footprint Capacitors_SMD:C_0603_HandSoldering -> Capacitors_SMD:C_0603
- C7: renamed from C8; footprint Capacitors_SMD:C_0603_HandSoldering -> Capacitors_SMD:C_0603
- C8: renamed from C9; footprint Capacitors_SMD:C_0603_HandSoldering -> Capacitors_SMD:C_0603
- C9: renamed from C3; value 1u -> 10u; footprint Capacitors_SMD:C_0603_HandSoldering -> Capacitors_SMD:C_0603
- D4: renamed from D2; footprint footprints:D_0603 -> Resistors_SMD:R_0603
- D5: renamed from D4; footprint footprints:D_0603 -> Resistors_SMD:R_0603
- FB1, FB2: footprint footprints:L_0603 -> Resistors_SMD:R_0603
- J2: renamed from J3; footprint footprints:FTSH-105-01-L-DV-K -> Pin_Headers:Pin_Header_Straight_2x05_Pitch1.27mm
- J4: footprint footprints:FTSH-105-01-L-DV-K -> Pin_Headers:Pin_Header_Straight_2x05_Pitch1.27mm
- R1: footprint Resistors_SMD:R_0603_HandSoldering -> Resistors_SMD:R_0603
- R10: renamed from R8; footprint Resistors_SMD:R_0603_HandSoldering -> Resistors_SMD:R_0603
- R11: renamed from R9; footprint Resistors_SMD:R_0603_HandSoldering -> Resistors_SMD:R_0603
- R12: renamed from R10; footprint Resistors_SMD:R_0603_HandSoldering -> Resistors_SMD:R_0603
- R13: renamed from R11; footprint Resistors_SMD:R_0603_HandSoldering -> Resistors_SMD:R_0603
- R4: renamed from R5; footprint Resistors_SMD:R_0603_HandSoldering -> Resistors_SMD:R_0603
- R5: renamed from R4; footprint Resistors_SMD:R_0603_HandSoldering -> Resistors_SMD:R_0603
- R8: renamed from R6; footprint Resistors_SMD:R_0603_HandSoldering -> Resistors_SMD:R_0603
- R9: renamed from R7; footprint Resistors_SMD:R_0603_HandSoldering -> Resistors_SMD:R_0603
- U1: footprint SMD_Packages:SSOP-14 -> footprints:DHVQFN14
- renumbered J6 to J3, J2 to J5, J5 to J6, JP2 to JP1, SW3 to SW2, SW2 to SW3, U5 to U4, U6 to U5
Connections:
- wire segments 207 -> 210
- no-connect marks 13 -> 17
Other:
- note added: "Optional Power Supply (DNP)"
- note added: "Target"
- note removed: "LDO"
- note removed: "Target SWD"
- note removed: "Target UART"
- moved on the sheet: C1, C10, C12, C13, C14, C15, C5, C6, C9, D4, D5, D6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

Commit message: progress
simplify LEDs
fix ferrite bead on 5v
lots of routing I'll have to redo anyway later
Parts:
- removed C2: 10u, Capacitors_SMD:C_0603, symbol C
- removed D7: D_Schottky, Diodes_SMD:SOD-523, symbol D_Schottky
- removed Q1, Q2, Q3: Q_NMOS_DGS, TO_SOT_Packages_SMD:SOT-23, symbol Q_NMOS_DGS
- removed R12, R13: 0, Resistors_SMD:R_0603, symbol R
- U1: renamed from U?; footprint (none) -> footprints:SOT457
- renumbered D4 to D1, D5 to D2, D6 to D3, R4 to R2, R5 to R3, R6 to R4, R7 to R5, R8 to R6, R9 to R7, R10 to R8, R11 to R9, U1 to U2, U2 to U3, U3 to U4, U4 to U5, U5 to U6
Connections:
- wire segments 210 -> 196
Other:
- note removed: "DNP"
- moved on the sheet: FB2, R7, R9
